File: z80_qfn64dip/z80_qfn64dip.kicad_sch (KiCad schematic)
At the start: 59 parts, among them J1 Conn_08, U1 Caravel_QFN, U2 Z80CPU, U3 TPS7A2033PDQNRM3, U4 TPS7A2018PDQNRM3, U5 TPS7A2050PDQNRM3, U6 AT25EU0081A, X1 10MHz

Commit message: Update mezzanine and Z80 QFN hardware designs
Parts:
- removed JP1: J_SDI, ProjectLibrary:SolderJumper-2_P2x0.9mm_Open_TrianglePad, symbol Jumper:SolderJumper_2_Open
- removed JP2: J_SCK, ProjectLibrary:SolderJumper-2_P2x0.9mm_Open_TrianglePad, symbol Jumper:SolderJumper_2_Open
- removed JP3: J_JTAG, ProjectLibrary:SolderJumper-2_P2x0.9mm_Open_TrianglePad, symbol Jumper:SolderJumper_2_Open
- removed JP4: J_SDO, ProjectLibrary:SolderJumper-2_P2x0.9mm_Open_TrianglePad, symbol Jumper:SolderJumper_2_Open
- added JP1: JSDI, ProjectLibrary:SolderJumper-2_P1.3mm_Bridged_RoundedPad1.0x1.5mm_Small_Margin, symbol Jumper:SolderJumper_2_Bridged
- added JP2: JSCK, ProjectLibrary:SolderJumper-2_P1.3mm_Bridged_RoundedPad1.0x1.5mm_Small_Margin, symbol Jumper:SolderJumper_2_Bridged
- added JP3: JJTAG, ProjectLibrary:SolderJumper-2_P1.3mm_Bridged_RoundedPad1.0x1.5mm_Small_Margin, symbol Jumper:SolderJumper_2_Bridged
- added JP5: JSDO, ProjectLibrary:SolderJumper-2_P1.3mm_Bridged_RoundedPad1.0x1.5mm_Small_Margin, symbol Jumper:SolderJumper_2_Bridged
- added TP14: RESET, ProjectLibrary:TestPoint_Pad_D1.0mm_Small_Margin, symbol Connector:TestPoint
- added TP15, TP16: GND, ProjectLibrary:TestPoint_Pad_D1.0mm_Small_Margin, symbol Connector:TestPoint
- R12: value 4k7 -> 10k
Connections:
- net GND: now also TP15.1, TP16.1
- net HK_JTAG: now also JP3.1 (A)
- net HK_SCK: now also JP2.1 (A)
- net HK_SDI: now also JP1.1 (A)
- net HK_SDO: now also JP5.2 (B)
- net ~{SOC_RST}: now also TP14.1
- net HKSDI: now reaches J1.8 (Pin_8)
- net HKSDI: now also JP1.2 (B)
- net HKSDO: now reaches J1.5 (Pin_5)
- net HKSDO: now also JP5.1 (A)
- net HKJTAG: now reaches J1.2 (Pin_2)
- net HKJTAG: now also JP3.2 (B)
- net HKSCK: now reaches J1.6 (Pin_6)
- net HKSCK: now also JP2.2 (B)
Other:
- moved on the sheet: C19, J1
